Commit message: changes

File: ur3_gripper_sim/urdf/ur3_gripper.urdf.xacro (robot description, xacro)
@@ -2,6 +2,6 @@
 <robot name="rg2" xmlns:xacro="http://www.ros.org/wiki/xacro">
     <xacro:property name="pi" value="3.141592654" />
-    <xacro:include filename="$(find rg2_description)/urdf/rg2.gazebo.xacro" />
-    <xacro:include filename="$(find rg2_description)/urdf/rg2.transmissions.xacro" />
+    <xacro:include filename="$(find ur3_gripper_sim)/urdf/ur3_gripper.gazebo.xacro" />
+    <xacro:include filename="$(find ur3_gripper_sim)/urdf/ur3_gripper.transmissions.xacro" />
     <link name="base_link">
     </link>
@@ -15,11 +15,11 @@
             <origin xyz="0.00 0.00 0.00" rpy="0.00 0.00 0.00"/>
             <geometry>
-                <mesh filename="package://rg2_description/meshes/collision/RG2_Hand_col.STL"/>
-            </geometry>
-        </collision>
-        <visual>
-            <origin xyz="0.00 0.00 0.00" rpy="0.00 0.00 0.00"/>
-            <geometry>
-                <mesh filename="package://rg2_description/meshes/visual/RG2_Hand_vis.STL"/>
+                <mesh filename="package://ur3_gripper_sim/meshes/collision/RG2_Hand_col.STL"/>
+            </geometry>
+        </collision>
+        <visual>
+            <origin xyz="0.00 0.00 0.00" rpy="0.00 0.00 0.00"/>
+            <geometry>
+                <mesh filename="package://ur3_gripper_sim/meshes/visual/RG2_Hand_vis.STL"/>
             </geometry>
         </visual>
@@ -55,11 +55,11 @@
             <origin xyz="0.00 0.00 0.00" rpy="0.00 0.00 0.00"/>
             <geometry>
-                <mesh filename="package://rg2_description/meshes/collision/RG2_LeftMomentArm_col.STL"/>
-            </geometry>
-        </collision>
-        <visual>
-            <origin xyz="0.00 0.00 0.00" rpy="0.00 0.00 0.00"/>
-            <geometry>
-                <mesh filename="package://rg2_description/meshes/visual/RG2_LeftMomentArm_vis.STL"/>
+                <mesh filename="package://ur3_gripper_sim/meshes/collision/RG2_LeftMomentArm_col.STL"/>
+            </geometry>
+        </collision>
+        <visual>
+            <origin xyz="0.00 0.00 0.00" rpy="0.00 0.00 0.00"/>
+            <geometry>
+                <mesh filename="package://ur3_gripper_sim/meshes/visual/RG2_LeftMomentArm_vis.STL"/>
             </geometry>
         </visual>
@@ -88,11 +88,11 @@
             <origin xyz="0.00 0.00 0.00" rpy="0.00 0.00 0.00"/>
             <geometry>
-                <mesh filename="package://rg2_description/meshes/collision/RG2_LeftFinger_col.STL"/>
-            </geometry>
-        </collision>
-        <visual>
-            <origin xyz="0.00 0.00 0.00" rpy="0.00 0.00 0.00"/>
-            <geometry>
-                <mesh filename="package://rg2_description/meshes/visual/RG2_LeftFinger_vis.STL"/>
+                <mesh filename="package://ur3_gripper_sim/meshes/collision/RG2_LeftFinger_col.STL"/>
+            </geometry>
+        </collision>
+        <visual>
+            <origin xyz="0.00 0.00 0.00" rpy="0.00 0.00 0.00"/>
+            <geometry>
+                <mesh filename="package://ur3_gripper_sim/meshes/visual/RG2_LeftFinger_vis.STL"/>
             </geometry>
         </visual>
@@ -121,11 +121,11 @@
             <origin xyz="0.00 0.00 0.00" rpy="0.00 0.00 0.00"/>
             <geometry>
-                <mesh filename="package://rg2_description/meshes/collision/RG2_LeftTrussArm_col.STL"/>
-            </geometry>
-        </collision>
-        <visual>
-            <origin xyz="0.00 0.00 0.00" rpy="0.00 0.00 0.00"/>
-            <geometry>
-                <mesh filename="package://rg2_description/meshes/visual/RG2_LeftTrussArm_vis.STL"/>
+                <mesh filename="package://ur3_gripper_sim/meshes/collision/RG2_LeftTrussArm_col.STL"/>
+            </geometry>
+        </collision>
+        <visual>
+            <origin xyz="0.00 0.00 0.00" rpy="0.00 0.00 0.00"/>
+            <geometry>
+                <mesh filename="package://ur3_gripper_sim/meshes/visual/RG2_LeftTrussArm_vis.STL"/>
             </geometry>
         </visual>
@@ -155,11 +155,11 @@
             <origin xyz="0.00 0.00 0.00" rpy="0.00 0.00 0.00"/>
             <geometry>
-                <mesh filename="package://rg2_description/meshes/collision/RG2_RightMomentArm_col.STL"/>
-            </geometry>
-        </collision>
-        <visual>
-            <origin xyz="0.00 0.00 0.00" rpy="0.00 0.00 0.00"/>
-            <geometry>
-                <mesh filename="package://rg2_description/meshes/visual/RG2_RightMomentArm_vis.STL"/>
+                <mesh filename="package://ur3_gripper_sim/meshes/collision/RG2_RightMomentArm_col.STL"/>
+            </geometry>
+        </collision>
+        <visual>
+            <origin xyz="0.00 0.00 0.00" rpy="0.00 0.00 0.00"/>
+            <geometry>
+                <mesh filename="package://ur3_gripper_sim/meshes/visual/RG2_RightMomentArm_vis.STL"/>
             </geometry>
         </visual>
@@ -188,11 +188,11 @@
             <origin xyz="0.00 0.00 0.00" rpy="0.00 0.00 0.00"/>
             <geometry>
-                <mesh filename="package://rg2_description/meshes/collision/RG2_RightFinger_col.STL"/>
-            </geometry>
-        </collision>
-        <visual>
-            <origin xyz="0.00 0.00 0.00" rpy="0.00 0.00 0.00"/>
-            <geometry>
-                <mesh filename="package://rg2_description/meshes/visual/RG2_RightFinger_vis.STL"/>
+                <mesh filename="package://ur3_gripper_sim/meshes/collision/RG2_RightFinger_col.STL"/>
+            </geometry>
+        </collision>
+        <visual>
+            <origin xyz="0.00 0.00 0.00" rpy="0.00 0.00 0.00"/>
+            <geometry>
+                <mesh filename="package://ur3_gripper_sim/meshes/visual/RG2_RightFinger_vis.STL"/>
             </geometry>
         </visual>
@@ -221,11 +221,11 @@
             <origin xyz="0.00 0.00 0.00" rpy="0.00 0.00 0.00"/>
             <geometry>
-                <mesh filename="package://rg2_description/meshes/collision/RG2_RightTrussArm_col.STL"/>
-            </geometry>
-        </collision>
-        <visual>
-            <origin xyz="0.00 0.00 0.00" rpy="0.00 0.00 0.00"/>
-            <geometry>
-                <mesh filename="package://rg2_description/meshes/visual/RG2_RightTrussArm_vis.STL"/>
+                <mesh filename="package://ur3_gripper_sim/meshes/collision/RG2_RightTrussArm_col.STL"/>
+            </geometry>
+        </collision>
+        <visual>
+            <origin xyz="0.00 0.00 0.00" rpy="0.00 0.00 0.00"/>
+            <geometry>
+                <mesh filename="package://ur3_gripper_sim/meshes/visual/RG2_RightTrussArm_vis.STL"/>
             </geometry>
         </visual>

Commit message: blah blah blah

File: ur3_gripper_sim/urdf/ur3_gripper.urdf.xacro (robot description, xacro)
@@ -4,11 +4,4 @@
     <xacro:include filename="$(find ur3_gripper_sim)/urdf/ur3_gripper.gazebo.xacro" />
     <xacro:include filename="$(find ur3_gripper_sim)/urdf/ur3_gripper.transmissions.xacro" />
-    <link name="base_link">
-    </link>
-    <joint name="base_fixed_joint" type="fixed">
-        <parent link="base_link"/>
-        <child link="hand_link"/>
-        <origin xyz="0.000 0.000 0.000" rpy="0 0 0"/>
-    </joint>
     <link name="hand_link">
         <collision>
